File: hardware/src_files/relay_logic_board.kicad_pcb (KiCad board)
At the start: 2 copper layers, 76 x 58 mm, 39 parts, among them J2 Screw_Terminal_01x07, J3 Screw_Terminal_01x09, J4 Conn_01x05, J5 Conn_02x03_Odd_Even, K1 G5LE-14, K2 G5LE-14, Q1 MMBT3904, Q2 MMBT3904, U1 ATmega328P-A, Y1 16MHz

Commit message: hardware files update, bom,gerbers&centroid files
hardware files update, bom,gerbers&centroid files
Parts:
- J2: footprint TerminalBlock_Phoenix:TerminalBlock_Phoenix_MPT-0,5-7-2.54_1x07_P2.54mm_Horizontal -> TerminalBlock_4Ucon:TerminalBlock_4Ucon_1x07_P3.50mm_Horizontal
- J3: footprint TerminalBlock_Phoenix:TerminalBlock_Phoenix_MPT-0,5-9-2.54_1x09_P2.54mm_Horizontal -> TerminalBlock_4Ucon:TerminalBlock_4Ucon_1x09_P3.50mm_Horizontal
- moved R1 5.64 mm to (133.0, 73.2)
- moved JP1 5.63 mm to (129.7, 70.5)
- moved K1 0.44 mm to (164.0, 95.1)
- moved Q1 0.38 mm to (170.6, 96.8)
- moved R11 0.33 mm to (170.5, 77.3)
- moved R10 0.32 mm to (170.4, 94.2)
- moved J2 0.16 mm to (161.2, 71.2)
- moved K2 0.15 mm to (164.1, 77.8)
- moved Q2 0.12 mm to (170.7, 79.8)
Connections:
- JP1 pad 3: Net-(JP1-Pad3) -> GND
Routing:
- net /ac_l: track 93.1 -> 102.8 mm
- net /ac_relay_2: track 47.2 -> 37.8 mm
- net +5V: track 215.0 -> 209.6 mm
- net /in1: track 83.4 -> 78.1 mm
- net Net-(J2-Pad5): track 45.0 -> 40.6 mm
- net GND: track 40.9 -> 44.3 mm
- net Net-(J2-Pad6): track 48.8 -> 46.9 mm, vias 1 -> 0
- net /ac_n: track 82.4 -> 84.1 mm
- net +24V: track 102.3 -> 103.8 mm
- net Net-(J2-Pad4): track 41.4 -> 40.0 mm
- net /ac_relay_1: track 12.2 -> 11.1 mm
- net /out1: track 98.3 -> 98.8 mm
Other:
- board text added: "+5V"
- board text added: "IN1"
